File: _autosave-planck.kicad_sch (KiCad schematic)
At the start: 53 parts, among them J1 USB_C_Receptacle_USB2.0, K1 KEYSW, K2 KEYSW, K3 KEYSW, K4 KEYSW, SW1 SW_PUSH, U1 ATmega32U4-M, Y1 Crystal_GND24_Small

Commit message: added basic layout
Parts:
- TP10: value TestPoint -> PB5
- TP11: value TestPoint -> PB6
- TP12: value TestPoint -> PB7
- TP13: value TestPoint -> PC6
- TP14: value TestPoint -> PC7
- TP15: value TestPoint -> PD0
- TP16: value TestPoint -> PD1
- TP17: value TestPoint -> PD2
- TP18: value TestPoint -> PD3
- TP19: value TestPoint -> PD4
- TP20: value TestPoint -> PD6
- TP21: value TestPoint -> PD7
- TP22: value TestPoint -> PE6
- TP23: value TestPoint -> PF6
- TP24: value TestPoint -> PF7
- TP3: value TestPoint -> AREF
- TP4: value TestPoint -> PD5
- TP5: value TestPoint -> PB0
- TP6: value TestPoint -> PB1
- TP7: value TestPoint -> PB2
- TP8: value TestPoint -> PB3
- TP9: value TestPoint -> PB4
Connections:
- net PE6: now reaches TP22.1, U1.1 (PE6)
- net PB2: now reaches TP7.1, U1.10 (PB2)
- net PB3: now reaches TP8.1, U1.11 (PB3)
- net PB7: now reaches TP12.1, U1.12 (PB7)
- net PD0: now reaches TP15.1, U1.18 (PD0)
- net PD1: now reaches TP16.1, U1.19 (PD1)
- net PD2: now reaches TP17.1, U1.20 (PD2)
- net PD3: now reaches TP18.1, U1.21 (PD3)
- net PD5: now reaches TP4.1, U1.22 (PD5)
- net PD4: now reaches TP19.1, U1.25 (PD4)
- net PD6: now reaches TP20.1, U1.26 (PD6)
- net PD7: now reaches TP21.1, U1.27 (PD7)
- net PB4: now reaches TP9.1, U1.28 (PB4)
- net PB5: now reaches TP10.1, U1.29 (PB5)
- net PB6: now reaches TP11.1, U1.30 (PB6)
- net PC6: now reaches TP13.1, U1.31 (PC6)
- net PC7: now reaches TP14.1, U1.32 (PC7)
- net PF7: now reaches TP24.1, U1.36 (PF7)
- net PF6: now reaches TP23.1, U1.37 (PF6)
- net PB0: now reaches TP5.1, U1.8 (PB0)
- net PB1: now reaches TP6.1, U1.9 (PB1)
- net reset renamed ~reset
