File: _autosave-planck.kicad_pcb (KiCad board)
At the start: 4 copper layers, 53 parts, among them J1 USB_C_Receptacle_USB2.0, K1 KEYSW, K2 KEYSW, K3 KEYSW, K4 KEYSW, SW1 SW_PUSH, U1 ATmega32U4-M, Y1 Crystal_GND24_Small

Commit message: poured gnd plane
Parts:
- moved TP14 58.4 mm to (91.9, 87.4)
- moved TP13 57.5 mm to (94.5, 87.4)
- moved TP23 56.2 mm to (86.9, 87.4)
- moved TP3 47.3 mm to (102.1, 87.4)
- moved TP19 45.9 mm to (91.9, 91.4)
- moved TP4 45.9 mm to (89.4, 91.4)
- moved TP10 45.9 mm to (89.4, 83.3)
- moved TP11 45.9 mm to (86.9, 83.3)
- moved TP12 45.9 mm to (84.3, 83.3)
- moved TP15 45.9 mm to (102.1, 91.4)
- moved TP16 45.9 mm to (99.6, 91.4)
- moved TP17 45.9 mm to (97.0, 91.4)
- moved TP18 45.9 mm to (94.5, 91.4)
- moved TP20 45.9 mm to (86.9, 91.4)
- moved TP21 45.9 mm to (84.3, 91.4)
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Changed lines of the file:
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@@
   )
   (footprint "Diode_SMD:D_SOD-123" (layer "F.Cu")
-    (at 87.376 112.014 180)
+    (at 87.376 112.014)
     (descr "SOD-123")
     (tags "SOD-123")
@@
     (fp_line (start -0.35 0) (end 0.25 -0.4) (layer "F.Fab") (width 0.1))
     (fp_line (start 0.25 0.4) (end -0.35 0) (layer "F.Fab") (width 0.1))
-    (pad "1" smd rect locked (at -1.65 0 180) (size 0.9 1.2) (layers "F.Cu" "F.Paste" "F.Mask")
+    (pad "1" smd rect locked (at -1.65 0) (size 0.9 1.2) (layers "F.Cu" "F.Paste" "F.Mask")
       (net 6 "/row0") (pinfunction "K") (pintype "passive"))
-    (pad "2" smd rect locked (at 1.65 0 180) (size 0.9 1.2) (layers "F.Cu" "F.Paste" "F.Mask")
+    (pad "2" smd rect locked (at 1.65 0) (size 0.9 1.2) (layers "F.Cu" "F.Paste" "F.Mask")
       (net 7 "Net-(D1-Pad2)") (pinfunction "A") (pintype "passive"))
     (model "${KICAD6_3DMODEL_DIR}/Diode_SMD.3dshapes/D_SOD-123.wrl"
@@
   )
   (footprint "TestPoint:TestPoint_Pad_D1.0mm" (layer "B.Cu")
-    (at 87.376 37.592 180)
+    (at 91.948 83.312 180)
     (descr "SMD pad as test Point, diameter 1.0mm")
     (tags "test point SMD pad")
@@
   )
   (footprint "TestPoint:TestPoint_Pad_D1.0mm" (layer "B.Cu")
-    (at 92.456 37.592 180)
+    (at 97.028 83.312 180)
     (descr "SMD pad as test Point, diameter 1.0mm")
     (tags "test point SMD pad")
@@
   )
   (footprint "Button_Switch_Keyboard:SW_Cherry_MX_1.00u_PCB" (layer "B.Cu")
-    (at 104.648 101.809 180)
+    (at 104.14 101.809 180)
     (descr "Cherry MX keyswitch, 1.00u, PCB mount, http://cherryamericas.com/wp-content/uploads/2014/12/mx_cat.pdf")
     (tags "Cherry MX keyswitch 1.00u PCB")
@@
   )
   (footprint "Button_Switch_Keyboard:SW_Cherry_MX_1.00u_PCB" (layer "B.Cu")
-    (at 84.328 101.809 180)
+    (at 84.836 101.809 180)
     (descr "Cherry MX keyswitch, 1.00u, PCB mount, http://cherryamericas.com/wp-content/uploads/2014/12/mx_cat.pdf")
     (tags "Cherry MX keyswitch 1.00u PCB")
@@
   )
   (footprint "TestPoint:TestPoint_Pad_D1.0mm" (layer "B.Cu")
-    (at 97.536 37.592 180)
+    (at 102.108 83.312 180)
     (descr "SMD pad as test Point, diameter 1.0mm")
     (tags "test point SMD pad")
@@
   )
   (footprint "TestPoint:TestPoint_Pad_D1.0mm" (layer "B.Cu")
-    (at 94.996 45.72 180)
+    (at 99.568 91.44 180)
     (descr "SMD pad as test Point, diameter 1.0mm")
     (tags "test point SMD pad")
@@
   )
   (footprint "TestPoint:TestPoint_Pad_D1.0mm" (layer "B.Cu")
-    (at 89.916 37.592 180)
+    (at 94.488 83.312 180)
     (descr "SMD pad as test Point, diameter 1.0mm")
     (tags "test point SMD pad")
@@
   )
   (footprint "TestPoint:TestPoint_Pad_D1.0mm" (layer "B.Cu")
-    (at 97.536 45.72 180)
+    (at 102.108 91.44 180)
     (descr "SMD pad as test Point, diameter 1.0mm")
     (tags "test point SMD pad")
@@
   )
   (footprint "TestPoint:TestPoint_Pad_D1.0mm" (layer "B.Cu")
-    (at 87.376 45.716 180)
+    (at 91.948 91.436 180)
     (descr "SMD pad as test Point, diameter 1.0mm")
     (tags "test point SMD pad")
@@
   )
   (footprint "TestPoint:TestPoint_Pad_D1.0mm" (layer "B.Cu")
-    (at 92.456 45.72 180)
+    (at 97.028 91.44 180)
     (descr "SMD pad as test Point, diameter 1.0mm")
     (tags "test point SMD pad")
@@
   )
   (footprint "TestPoint:TestPoint_Pad_D1.0mm" (layer "B.Cu")
-    (at 79.756 45.72 180)
+    (at 84.328 91.44 180)
     (descr "SMD pad as test Point, diameter 1.0mm")
     (tags "test point SMD pad")
@@
   )
   (footprint "TestPoint:TestPoint_Pad_D1.0mm" (layer "B.Cu")
-    (at 96.516 49.812 180)
+    (at 89.408 87.376 180)
     (descr "SMD pad as test Point, diameter 1.0mm")
     (tags "test point SMD pad")
@@
   )
   (footprint "TestPoint:TestPoint_Pad_D1.0mm" (layer "B.Cu")
-    (at 109.22 40.64 180)
+    (at 102.108 87.376 180)
     (descr "SMD pad as test Point, diameter 1.0mm")
     (tags "test point SMD pad")
@@
   )
   (footprint "TestPoint:TestPoint_Pad_D1.0mm" (layer "B.Cu")
-    (at 107.186 31.016 180)
+    (at 91.948 87.376 180)
     (descr "SMD pad as test Point, diameter 1.0mm")
     (tags "test point SMD pad")
@@
   )
   (footprint "TestPoint:TestPoint_Pad_D1.0mm" (layer "B.Cu")
-    (at 83.314 30.984 180)
+    (at 94.488 87.376 180)
     (descr "SMD pad as test Point, diameter 1.0mm")
     (tags "test point SMD pad")
@@
   )
   (footprint "TestPoint:TestPoint_Pad_D1.0mm" (layer "B.Cu")
-    (at 82.296 37.592 180)
+    (at 86.868 83.312 180)
     (descr "SMD pad as test Point, diameter 1.0mm")
     (tags "test point SMD pad")
@@
   )
   (footprint "TestPoint:TestPoint_Pad_D1.0mm" (layer "B.Cu")
-    (at 82.294 50.828 180)
+    (at 84.326 87.404 180)
     (descr "SMD pad as test Point, diameter 1.0mm")
     (tags "test point SMD pad")
@@
   )
   (footprint "Button_Switch_Keyboard:SW_Cherry_MX_1.00u_PCB" (layer "B.Cu")
-    (at 104.648 121.92 180)
+    (at 104.14 121.158 180)
     (descr "Cherry MX keyswitch, 1.00u, PCB mount, http://cherryamericas.com/wp-content/uploads/2014/12/mx_cat.pdf")
     (tags "Cherry MX keyswitch 1.00u PCB")
@@
   )
   (footprint "TestPoint:TestPoint_Pad_D1.0mm" (layer "B.Cu")
-    (at 79.756 37.592 180)
+    (at 84.328 83.312 180)
     (descr "SMD pad as test Point, diameter 1.0mm")
     (tags "test point SMD pad")
@@
   )
   (footprint "Button_Switch_Keyboard:SW_Cherry_MX_1.00u_PCB" (layer "B.Cu")
-    (at 84.328 122.009 180)
+    (at 84.836 121.158 180)
     (descr "Cherry MX keyswitch, 1.00u, PCB mount, http://cherryamericas.com/wp-content/uploads/2014/12/mx_cat.pdf")
     (tags "Cherry MX keyswitch 1.00u PCB")
@@
   )
   (footprint "TestPoint:TestPoint_Pad_D1.0mm" (layer "B.Cu")
-    (at 84.836 37.592 180)
+    (at 89.408 83.312 180)
     (descr "SMD pad as test Point, diameter 1.0mm")
     (tags "test point SMD pad")
@@
   )
   (footprint "TestPoint:TestPoint_Pad_D1.0mm" (layer "B.Cu")
-    (at 84.836 45.716 180)
+    (at 89.408 91.436 180)
     (descr "SMD pad as test Point, diameter 1.0mm")
     (tags "test point SMD pad")
@@
   )
   (footprint "TestPoint:TestPoint_Pad_D1.0mm" (layer "B.Cu")
-    (at 107.696 44.704 180)
+    (at 97.028 87.376 180)
     (descr "SMD pad as test Point, diameter 1.0mm")
     (tags "test point SMD pad")
@@
   )
   (footprint "TestPoint:TestPoint_Pad_D1.0mm" (layer "B.Cu")
-    (at 82.296 45.72 180)
+    (at 86.868 91.44 180)
     (descr "SMD pad as test Point, diameter 1.0mm")
     (tags "test point SMD pad")
@@
   )
   (footprint "TestPoint:TestPoint_Pad_D1.0mm" (layer "B.Cu")
-    (at 110.236 44.704 180)
+    (at 99.568 87.376 180)
     (descr "SMD pad as test Point, diameter 1.0mm")
     (tags "test point SMD pad")
@@
   )
   (footprint "TestPoint:TestPoint_Pad_D1.0mm" (layer "B.Cu")
-    (at 89.916 45.72 180)
+    (at 94.488 91.44 180)
     (descr "SMD pad as test Point, diameter 1.0mm")
     (tags "test point SMD pad")
@@
   )
   (footprint "TestPoint:TestPoint_Pad_D1.0mm" (layer "B.Cu")
-    (at 94.996 37.592 180)
+    (at 99.568 83.312 180)
     (descr "SMD pad as test Point, diameter 1.0mm")
     (tags "test point SMD pad")
@@
   )
   (footprint "TestPoint:TestPoint_Pad_D1.0mm" (layer "B.Cu")
-    (at 92.456 31.496 180)
-    (descr "SMD pad as test Point, diameter 1.0mm")
-    (tags "test point SMD pad")
+    (at 86.868 87.376 180)
+    (descr "SMD pad as test Point, diameter 1.0mm")
+    (tags "test point SMD pad")
